File: PCB/PCB.kicad_pcb (KiCad board)
At the start: 2 copper layers, 360.5 x 286.5 mm, 52 parts, among them SW1 SW_Push, SW10 SW_Push, SW11 SW_Push, SW12 SW_Push, SW13 SW_Push, SW14 SW_Push, SW15 SW_Push, SW16 SW_Push, SW17 SW_Push, SW2 SW_Push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

Commit message: finished pcb + firmware
Parts:
- added J1: Conn_02x06_Counter_Clockwise, Connector_PinHeader_2.54mm:PinHeader_2x06_P2.54mm_Vertical, F.Cu at (129.3, 35.5)
- added J2: Conn_02x06_Counter_Clockwise, Connector_PinHeader_2.54mm:PinHeader_2x06_P2.54mm_Vertical, F.Cu at (225.7, 75.5)
- U1: moved to B.Cu
- moved U1 117.9 mm to (226.9, 84.6), turned to 180 degrees
- moved D17 19.9 mm to (161.7, 102.4), turned to 0 degrees
- moved D12 15.7 mm to (161.7, 95.2), turned to 0 degrees
- moved D8 15.2 mm to (161.7, 72.6), turned to 0 degrees
- moved D4 14.7 mm to (161.7, 52.4), turned to 0 degrees
Connections:
- U1 pad 1: COL0 -> COL0_MCU
- U1 pad 10: ROW1 -> ROW1_MCU
- U1 pad 11: ROW0 -> ROW0_MCU
- U1 pad 13: GND -> GND2
- U1 pad 14: +5V -> +5V-B
- U1 pad 2: COL1 -> COL1_MCU
- U1 pad 3: COL2 -> COL2_MCU
- U1 pad 4: COL3 -> COL3_MCU
- U1 pad 5: COL4 -> COL4_MCU
- U1 pad 7: LED -> LED_MCU
- U1 pad 8: ROW3 -> ROW3_MCU
- U1 pad 9: ROW2 -> ROW2_MCU
Routing:
- net +5V: track 0.00 -> 399.3 mm, vias 0 -> 1
- net ROW3: track 0.00 -> 149.1 mm, vias 0 -> 2
- net ROW2: track 0.00 -> 117.0 mm, vias 0 -> 1
- net COL0: track 0.00 -> 116.1 mm
- net COL1: track 0.00 -> 108.2 mm
- net ROW1: track 0.00 -> 105.0 mm, vias 0 -> 3
- net COL3: track 0.00 -> 98.3 mm
- net COL4: track 0.00 -> 98.3 mm, vias 0 -> 2
- net COL2: track 0.00 -> 95.6 mm
- net ROW0: track 0.00 -> 82.2 mm, vias 0 -> 1
- net LED: track 0.00 -> 50.9 mm
- net Net-(D28-DOUT): track 0.00 -> 39.3 mm
- net Net-(D29-DOUT): track 0.00 -> 32.4 mm
- net Net-(D19-DOUT): track 0.00 -> 31.1 mm
- net Net-(D24-DOUT): track 0.00 -> 27.1 mm
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- added copper zone on B.Cu, net GND2
- added copper zone on F.Cu, net GND2
Other:
- board size 360.5 x 286.5 mm -> 151.1 x 87.3 mm

Commit message: added cad files and gerbers
Parts:
- J1, J2: moved to B.Cu
- moved J1 2.57 mm to (131.9, 35.5), turned to 180 degrees
- moved J2 2.55 mm to (228.2, 75.5), turned to 180 degrees
Routing:
- net COL4: track 98.3 -> 84.8 mm
- net ROW3: track 149.1 -> 139.5 mm, vias 2 -> 0
- net GND2: track 16.3 -> 6.80 mm, vias 16 -> 34
- net LED: track 50.9 -> 42.8 mm, vias 0 -> 4
- net ROW0: track 82.2 -> 77.0 mm, vias 1 -> 0
- net COL1: track 108.2 -> 111.9 mm
- net COL2: track 95.6 -> 92.1 mm
- net COL0: track 116.1 -> 119.5 mm
- net +5V: track 399.3 -> 396.2 mm, vias 1 -> 2
- net COL2_MCU: track 9.61 -> 6.70 mm
- net COL0_MCU: track 9.41 -> 6.70 mm
- net COL3_MCU: track 9.41 -> 6.70 mm
- net COL1_MCU: track 9.41 -> 6.70 mm
- net COL4_MCU: track 9.41 -> 6.70 mm
- net +5V-B: track 9.49 -> 6.80 mm
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