File: PCB/PCB.kicad_sch (KiCad schematic)
At the start: 52 parts, among them SW1 SW_Push, SW10 SW_Push, SW11 SW_Push, SW12 SW_Push, SW13 SW_Push, SW14 SW_Push, SW15 SW_Push, SW16 SW_Push, SW17 SW_Push, SW2 SW_Push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

Commit message: finished pcb + firmware
Parts:
- added J1, J2: Conn_02x06_Counter_Clockwise, Connector_PinHeader_2.54mm:PinHeader_2x06_P2.54mm_Vertical, symbol Connector_Generic:Conn_02x06_Odd_Even
Connections:
- net +5V: now also J1.2 (Pin_2); no longer U1.14 (5V)
- net COL0: now also J1.1 (Pin_1); no longer U1.1 (PA02_A0_D0)
- net COL1: now also J1.3 (Pin_3); no longer U1.2 (PA4_A1_D1)
- net COL2: now also J1.5 (Pin_5); no longer U1.3 (PA10_A2_D2)
- net COL3: now also J1.7 (Pin_7); no longer U1.4 (PA11_A3_D3)
- net COL4: now also J1.9 (Pin_9); no longer U1.5 (PA8_A4_D4_SDA)
- net GND: now also J1.4 (Pin_4); no longer U1.13 (GND)
- net LED: now also J1.11 (Pin_11); no longer U1.7 (PB08_A6_D6_TX)
- net ROW0: now also J1.6 (Pin_6); no longer U1.11 (PA6_A10_D10_MOSI)
- net ROW1: now also J1.8 (Pin_8); no longer U1.10 (PA5_A9_D9_MISO)
- net ROW2: now also J1.10 (Pin_10); no longer U1.9 (PA7_A8_D8_SCK)
- net ROW3: now also J1.12 (Pin_12); no longer U1.8 (PB09_A7_D7_RX)
- new net +5V-B: J2.2 (Pin_2), U1.14 (5V)
- new net COL0_MCU: J2.1 (Pin_1), U1.1 (PA02_A0_D0)
- new net COL1_MCU: J2.3 (Pin_3), U1.2 (PA4_A1_D1)
- new net COL2_MCU: J2.5 (Pin_5), U1.3 (PA10_A2_D2)
- new net COL3_MCU: J2.7 (Pin_7), U1.4 (PA11_A3_D3)
- new net COL4_MCU: J2.9 (Pin_9), U1.5 (PA8_A4_D4_SDA)
- new net GND2: J2.4 (Pin_4), U1.13 (GND)
- new net LED_MCU: J2.11 (Pin_11), U1.7 (PB08_A6_D6_TX)
- new net ROW0_MCU: J2.6 (Pin_6), U1.11 (PA6_A10_D10_MOSI)
- new net ROW1_MCU: J2.8 (Pin_8), U1.10 (PA5_A9_D9_MISO)
- new net ROW2_MCU: J2.10 (Pin_10), U1.9 (PA7_A8_D8_SCK)
- new net ROW3_MCU: J2.12 (Pin_12), U1.8 (PB09_A7_D7_RX)

Commit message: added cad files and gerbers
Other:
- moved on the sheet: D1, D10, D11, D12, D13, D14, D15, D16, D17, D18, D19, D2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
